File: pcb/my-keeb.kicad_pcb (KiCad board)
At the start: 2 copper layers, 310 x 105 mm, 6 parts

Commit message: Update layout to 98% ISO Italian (100 keys with numpad and F-row)
Parts:
- added ?: , MountingHole:MountingHole_2.2mm_M2, F.Cu at (95.0, 65.0)
- added ?: , MountingHole:MountingHole_2.2mm_M2, F.Cu at (285.0, 65.0)
- moved ? 74.3 mm to (375.0, 125.0)
- moved ? 70.0 mm to (375.0, 5.00)
- moved ? 37.2 mm to (190.0, 65.0)
- moved ? 35.0 mm to (190.0, 2.00)
- moved ? 25.0 mm to (5.00, 125.0)
Other:
- board size 310 x 105 mm -> 380 x 130 mm
Changed lines of the file:
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@@
   (paper "A3")
   (title_block
-    (title "my-keeb — 65% ISO Italian Layout")
+    (title "my-keeb — 98% ISO Italian Layout")
     (date "2026-06-19")
-    (rev "1.0")
-    (comment 1 "68-key ISO IT, Cherry MX, ATmega32U4, USB-C")
+    (rev "2.0")
+    (comment 1 "100-key ISO IT 98%, Cherry MX, ATmega32U4, USB-C")
   )
   (layers
@@
   (net 4 "ROW3")
   (net 5 "ROW4")
-  (net 6 "COL0")
-  (net 7 "COL1")
-  (net 8 "COL2")
-  (net 9 "COL3")
-  (net 10 "COL4")
-  (net 11 "COL5")
-  (net 12 "COL6")
-  (net 13 "COL7")
-  (net 14 "COL8")
-  (net 15 "COL9")
-  (net 16 "COL10")
-  (net 17 "COL11")
-  (net 18 "COL12")
-  (net 19 "COL13")
-  (net 20 "COL14")
-  (net 21 "VCC")
-  (net 22 "GND")
-  (net 23 "D+")
-  (net 24 "D-")
-  ; PCB outline — 65% keyboard ~310mm x 105mm
-  (gr_line (start 0 0) (end 310 0) (layer "Edge.Cuts") (width 0.15))
-  (gr_line (start 310 0) (end 310 105) (layer "Edge.Cuts") (width 0.15))
-  (gr_line (start 310 105) (end 0 105) (layer "Edge.Cuts") (width 0.15))
-  (gr_line (start 0 105) (end 0 0) (layer "Edge.Cuts") (width 0.15))
+  (net 6 "ROW5")
+  (net 7 "COL0")
+  (net 8 "COL1")
+  (net 9 "COL2")
+  (net 10 "COL3")
+  (net 11 "COL4")
+  (net 12 "COL5")
+  (net 13 "COL6")
+  (net 14 "COL7")
+  (net 15 "COL8")
+  (net 16 "COL9")
+  (net 17 "COL10")
+  (net 18 "COL11")
+  (net 19 "COL12")
+  (net 20 "COL13")
+  (net 21 "COL14")
+  (net 22 "COL15")
+  (net 23 "COL16")
+  (net 24 "COL17")
+  (net 25 "COL18")
+  (net 26 "VCC")
+  (net 27 "GND")
+  (net 28 "D+")
+  (net 29 "D-")
+  ; PCB outline — 98% keyboard ~380mm x 130mm
+  (gr_line (start 0 0) (end 380 0) (layer "Edge.Cuts") (width 0.15))
+  (gr_line (start 380 0) (end 380 130) (layer "Edge.Cuts") (width 0.15))
+  (gr_line (start 380 130) (end 0 130) (layer "Edge.Cuts") (width 0.15))
+  (gr_line (start 0 130) (end 0 0) (layer "Edge.Cuts") (width 0.15))
   ; Mounting holes — M2 standoffs
   (footprint "MountingHole:MountingHole_2.2mm_M2" (at 5 5) (layer "F.Cu") (uuid "mh1"))
-  (footprint "MountingHole:MountingHole_2.2mm_M2" (at 305 5) (layer "F.Cu") (uuid "mh2"))
-  (footprint "MountingHole:MountingHole_2.2mm_M2" (at 5 100) (layer "F.Cu") (uuid "mh3"))
-  (footprint "MountingHole:MountingHole_2.2mm_M2" (at 305 100) (layer "F.Cu") (uuid "mh4"))
-  (footprint "MountingHole:MountingHole_2.2mm_M2" (at 155 52.5) (layer "F.Cu") (uuid "mh5"))
+  (footprint "MountingHole:MountingHole_2.2mm_M2" (at 375 5) (layer "F.Cu") (uuid "mh2"))
+  (footprint "MountingHole:MountingHole_2.2mm_M2" (at 5 125) (layer "F.Cu") (uuid "mh3"))
+  (footprint "MountingHole:MountingHole_2.2mm_M2" (at 375 125) (layer "F.Cu") (uuid "mh4"))
+  (footprint "MountingHole:MountingHole_2.2mm_M2" (at 190 65) (layer "F.Cu") (uuid "mh5"))
+  (footprint "MountingHole:MountingHole_2.2mm_M2" (at 95 65) (layer "F.Cu") (uuid "mh6"))
+  (footprint "MountingHole:MountingHole_2.2mm_M2" (at 285 65) (layer "F.Cu") (uuid "mh7"))
   ; USB-C connector — top center
-  (footprint "Connector_USB:USB_C_Receptacle_GCT_USB4085" (at 155 2) (layer "F.Cu") (uuid "usbc1"))
+  (footprint "Connector_USB:USB_C_Receptacle_GCT_USB4085" (at 190 2) (layer "F.Cu") (uuid "usbc1"))
 )
